File: ball_butler_circuit_diagram/Power and CAN.kicad_sch (KiCad schematic)
At the start: 12 parts

Commit message: Update schematic
Connections:
- net at U?. (GND): now also U?. (GND); no longer U?. (GND) (x5)
- net at U?. (GND): no longer U?. (GND)
- net at U?. (GND): now also U?. (GND), U?. (GND); no longer U?. (GND)
- new net: U?. (GND), U?. (GND), U?. (GND), U?. (GND), U?. (GND), U?. (GND), U?. (GND), U?. (GND), U?. (GND), U?. (GND)
- new net: U?. (GND), U?. (GND), U?. (GND), U?. (GND), U?. (GND), U?. (GND), U?. (GND), U?. (GND)
- new net: U?. (GND), U?. (GND) (x23)
- new net: U?. (GND), U?. (GND), U?. (GND) (x2)
- now unconnected: U?. (GND), U?. (GND), U?. (GND), U?. (GND), U?. (GND)
Other:
- note removed: "Commissioning checklist (fast) Power at 24-25 V. Enable S1 brake-resistor control + voltage feedback; set ramp-end ≤ 30.5 V. ODrive Documentation Fit the PSU series diode. ODrive Documentation Log during your worst throw/brake: vbus_voltage, axis*.motor.current_control.Ibus (regen is negative). Ensure vbus_voltage never exceeds ~30.5 V and adjust max_regen_current/ramp start-end as needed"
Changed lines of the file:
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@@
     (effects (font (size 1.5 1.5)) (justify left bottom))
-  )
-  (text "Commissioning checklist (fast)\n\nPower at 24-25 V.\n\nEnable S1 brake-resistor control + voltage feedback; set ramp-end ≤ 30.5 V. \nODrive Documentation\n\nFit the PSU series diode. \nODrive Documentation\n\nLog during your worst throw/brake: vbus_voltage, axis*.motor.current_control.Ibus (regen is negative). Ensure vbus_voltage never exceeds ~30.5 V and adjust max_regen_current/ramp start-end as needed"
-    (at 16.51 -8.89 0)
-    (effects (font (size 1.27 1.27)) (justify left bottom))
   )
   (text "<-- Approx. 1.5m long -->" (at 142.748 142.748 0)
