File: ball_butler_circuit_diagram/ball_butler_circuit_diagram.kicad_sch (KiCad schematic)
At the start: 16 parts

Commit message: Update schematic
Connections:
- net at U?. (NC): now also U?. (VIN)
- new net: U?. (GND), U?. (GND) (x3)
- new net: M?. (C), U?. (VIN) (x4)
- new net: U?. (PIN), U?. (VIN)
- new net: M?. (PWR2), U?. (VIN)
- new net: U?. (NC), U?. (VIN) (x4)
