File: ball_butler_circuit_diagram/programming_logic.kicad_sch (KiCad schematic)
At the start: 8 parts

Commit message: Update schematic
Connections:
- net at U?. (Measured_Yaw_Angle): now also U?. (Throw_Vel); no longer U?. (Reload_Yaw_Angle)
- net at U?. (Throw_Info): no longer U?. (Reload_Yaw_Angle)
- new net: U?. (Reload_Yaw_Angle), U?. (Target_Yaw_Angle), U?. (Yaw_Angle)
- new net: U?. (Measured_Yaw_Angle), U?. (Reload_Yaw_Angle) (x2)
- new net: U?. (Reload_Yaw_Angle), U?. (Throw_Info)
- new net: U?. (Reload_Yaw_Angle), U?. (Throw_Vel)
- new net: U?. (Measured_Yaw_Angle), U?. (Yaw_Angle) (x4)
- new net: U?. (Throw_Vel), U?. (Yaw_Angle) (x2)
- new net: U?. (Measured_Yaw_Angle), U?. (Target_Yaw_Angle)
